File: Escorna_botoneira_2_0/Escorna_Shield_botoneira_2_0B.sch (EAGLE design)
At the start: 22 parts, among them J1 22-27-2051-05, J2 22-27-2021-02

Commit message: Esquema actualizado
Parts:
- RT.7: value 10K -> 1K
Other:
- note added: "Aux. Connector"
- note added: "Backward"
- note added: "Botoneira 2.0"
- note added: "Buton Keys"
- note added: "Button keys"
- note added: "Connector to other CPUs"
- note added: "Escornabot CPU1.0 connector"
- note added: "Forward"
- note added: "Go"
- note added: "Led on board"
- note added: "Left"
- note added: "Reset"
- note added: "Right"
- note added: "S7"
- note added: "Shield Botoneira con Pull-up no Arduino"
- note added: "Teclas"
- note added: "Voltage Selector for J1 connector"
- note removed: "Atrás"
- note removed: "Botoneira con Pull-up no Arduino"
- note removed: "Botoneira versión 2.X"
- note removed: "De Fronte"
- note removed: "Dereita"
- note removed: "Esquerda"
- note removed: "IR"
- note removed: "Selector de tensión para conector de (A1.2.3)"
- moved on the sheet: J1-1, J1-2, J1-3, J1-4, J1-5, J2-1, J2-2, LED5MM, RT.1, RT.2, RT.3, RT.4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
