File: Escorna_botoneira_2_0/Escorna_Shield_botoneira_2_0B.brd (EAGLE design)
At the start: 50.2 x 50.2 mm, 24 parts, among them J1 22-27-2051-05, J2 22-27-2021-02

Commit message: Melloras
Melloras Botoneira a 2.0C
CPU a 1.01
Parts:
- D1: value (none) -> 3 a 5mm
- RT.7: value 10K -> 1K
- renumbered LED5MM to D1
