File: Escorna_botoneira_2_0/Escorna_Shield_botoneira_2_0C.sch (EAGLE design)
At the start: 22 parts, among them J1 22-27-2051-05, J2 22-27-2021-02

Commit message: Melloras
Melloras Botoneira a 2.0C
CPU a 1.01
Parts:
- removed H1: MOUNT-HOLE3.0, holes:MOUNT-HOLE3.0
- added J3: 22-05-7038-03, con-molex:22-05-7038-03
- added U$10: XDESIG, xdesig:XDESIG
- added U$3: XDESIG21, xdesig:XDESIG21
- added U$4, U$5, U$6, U$7: FRECHA, escorna:FRECHA
- added U$8: GO, escorna:GO
- added U$9: CANCELA, escorna:CANCELA
- J1: value 22-27-2051-05 -> (none); device con-molex:22-27-2051-05 -> con-lsta:FE13-1
- J2: value 22-27-2021-02 -> 22-05-7028-02; device con-molex:22-27-2021-02 -> con-molex:22-05-7028-02
- LED5MM: value 3 a 5mm -> (none)
- renumbered D1 to LED5MM
Connections:
- removed net LED1: ESSH1.A1_D11_D16, J1-2.S
- removed net LED2: ESSH1.A2_D12_D14, J1-3.S
- removed net LED3: ESSH1.A3_D13_D15, J1-4.S
- removed net N$11: RT.3.1, RT.4.2, S3.P, S3.P1
- removed net N$12: RT.4.1, RT.5.2, S4.P, S4.P1
- new net 3V3: ESSH1.3V3N, J1.11
- new net A0: ESSH1.A0_D10_D10, J1.9
- new net A1: ESSH1.A1_D11_D16, J1.8
- new net A2: ESSH1.A2_D12_D14, J1.7
- new net A3: ESSH1.A3_D13_D15, J1.6
- new net A6: ESSH1.A6_A2_A2, J1.3
- new net A7: ESSH1.A7_A3_A3, J1.2
- new net AREF: ESSH1.AREFN, J1.10
- new net D11: ESSH1.D11N, J3-1.S
- new net D12: ESSH1.D12N, J3-2.S
- new net D13: ESSH1.D13N, J1.12
- new net N$3: RT.2.2, S1.P1
- new net N$4: RT.1.1, S1.P
- new net N$5: RT.5.2, S4.P1
- new net N$8: RT.3.1, RT.4.2, S3.P
- new net N$9: RT.2.1, S2.P
- net A4: now also ESSH1.KEY/A4_A0_A0, J2-2.S; no longer ESSH1.A4_A0_A0, J2-1.S
- net GND: now also J1.13, J2-1.S, J3-3.S; no longer J1-1.S, J2-2.S
- net N$10: no longer RT.2.1, S2.P
- net N$13: no longer S5.P
- net N$2: now also J1.1; no longer J1-5.S
- net N$7: now also RT.4.1, S4.P; no longer RT.1.1, RT.2.2, S1.P, S1.P1
- net RST: no longer S7.P1
Other:
- note added: "000.C"
- note added: "Aux. Connectors"
- note added: "Clear"
- note added: "Keypad"
- note added: "Micro pro"
- note added: "Mini"
- note added: "Nano"
- note removed: "000.B"
- note removed: "Aux. Connector"
- note removed: "Buton Keys"
- note removed: "Button keys"
- note removed: "Teclas"
- note removed: "X"
- moved on the sheet: J2-1, J2-2, SJ1
