File: Escorna_botoneira_2_0/Escorna_Shield_botoneira_2_0D.sch (EAGLE design)
At the start: 31 parts, among them J2 22-05-7028-02, J3 22-05-7038-03, J4 22-05-7028-02

Commit message: Versión 2.0D
Other:
- note added: "Creative Commons Attribution-ShareAlike 4.0 International (CC BY-SA 4.0)"
- note removed: "Creative Commons Recoñecemento 4.0 Internacional (CC BY 4.0)"
Changed lines of the file:
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@@
 <wire x1="66.04" y1="86.36" x2="66.04" y2="83.82" width="0.1524" layer="97" style="shortdash"/>
 <text x="223.52" y="60.96" size="1.778" layer="97">90º rotate</text>
-<text x="170.688" y="29.21" size="2.1844" layer="97">Creative Commons Recoñecemento 4.0 Internacional (CC BY 4.0)</text>
+<text x="164.592" y="28.448" size="2.1844" layer="97">Creative Commons Attribution-ShareAlike 4.0 International (CC BY-SA 4.0)</text>
 </plain>
 <instances>
