File: Escorna_CPU_1_0/Escorna_CPU_1_01.brd (EAGLE design)
At the start: 50 x 50 mm, 28 parts, among them IC1 ULN2803, X3 22-23-2031

Commit message: Melloras
Melloras Botoneira a 2.0C
CPU a 1.01
Parts:
- moved U$1 29.4 mm to (13.5, 43.8)
- moved U$3 24.8 mm to (23.1, 21.5)
Routing:
- net GND: track 63.0 -> 82.5 mm
Other:
- board text added: "1.01"
- board text added: "Mot. Left"
- board text added: "Mot. Right"
- board text added: "XDeSIG 1506"
- board text added: "http://escornabot.com"
- board text removed: "1.0"
- board text removed: "1506"
- board text removed: "EscornaBot"
- board text removed: "EscornaBot 1.0"
- board text removed: "MOT. DER"
- board text removed: "MOT. ESQ"

Commit message: Xdesig update 2015-06-04
Parts:
- removed JP1: (no value), jumper:JP2
- added S2: (no value), escorna:SK-12F14-G
- U$6: device xdesig:XDESIG_CU -> xdesig:XDESIG_CU_2
- moved X4 0.19 mm to (3.17, 9.53)
Connections:
- removed net N$4: JP1.1, JP1.2, X4.2
- new net N$3: S2.P$3, X4.2
- net GND: now also S2.P$4, S2.P$5
- net RAW: now also S2.P$1, S2.P$2; no longer JP1.3
Routing:
- net N$4: track 7.08 -> 0.00 mm
- net N$3: track 0.00 -> 5.70 mm
- net RAW: track 90.2 -> 94.6 mm
- net GND: track 82.5 -> 81.9 mm
Changed lines of the file:
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@@
 <layers>
 <layer number="1" name="Top" color="1" fill="1" visible="no" active="yes"/>
-<layer number="16" name="Bottom" color="4" fill="1" visible="yes" active="yes"/>
+<layer number="16" name="Bottom" color="4" fill="1" visible="no" active="yes"/>
 <layer number="17" name="Pads" color="2" fill="1" visible="yes" active="yes"/>
 <layer number="18" name="Vias" color="2" fill="1" visible="yes" active="yes"/>
@@
 <text x="6.7945" y="36.449" size="1.27" layer="21" rot="R180">RESET</text>
 <text x="6.223" y="24.0665" size="0.8128" layer="21" rot="R180">TECLADO</text>
-<text x="6.985" y="0.1905" size="0.8128" layer="21">ON</text>
-<text x="0.127" y="1.2065" size="2.54" layer="21">+</text>
+<text x="14.7955" y="1.397" size="0.8128" layer="21">ON</text>
+<text x="1.016" y="3.302" size="2.54" layer="21">+</text>
 <text x="44.958" y="3.1115" size="1.016" layer="21" rot="R270">Tx</text>
 <text x="43.688" y="1.7145" size="1.016" layer="21" rot="R90">Rx</text>
@@
 <text x="23.4315" y="38.735" size="1.016" layer="21">D11</text>
 <text x="23.495" y="41.275" size="1.016" layer="21">D12</text>
-<text x="11.43" y="3.556" size="1.016" layer="21">Raw</text>
+<text x="14.0335" y="3.4925" size="1.016" layer="21">Raw</text>
 <text x="14.6685" y="8.255" size="1.016" layer="21">G</text>
 <text x="14.732" y="10.8585" size="1.016" layer="21">RST</text>
@@
 <wire x1="17.78" y1="41.91" x2="19.05" y2="41.91" width="0.254" layer="21" style="shortdash"/>
 <wire x1="19.05" y1="41.91" x2="19.05" y2="35.56" width="0.254" layer="21" style="shortdash"/>
-<text x="28.448" y="1.778" size="1.27" layer="16" font="vector" rot="MR0">XDeSIG 1506</text>
+<text x="39.243" y="31.9405" size="1.27" layer="16" font="vector" rot="MR270">XDeSIG 1506</text>
 <text x="26.035" y="13.5255" size="1.016" layer="22" rot="MR0">Gnd</text>
 <text x="26.035" y="15.9385" size="1.016" layer="22" rot="MR0">D2</text>
@@
 </autorouter>
 <elements>
-<element name="X4" library="con-ptr500" package="AK500/2" value="" x="3.175" y="9.3345" smashed="yes" rot="R270">
-<attribute name="NAME" x="5.3975" y="9.4615" size="1.016" layer="25" ratio="10"/>
-<attribute name="VALUE" x="-2.54" y="14.4145" size="1.778" layer="27" ratio="10" rot="R270"/>
-<attribute name="OC_NEWARK" value="unknown" x="3.175" y="9.3345" size="1.778" layer="27" rot="R270" display="off"/>
-<attribute name="MPN" value="" x="3.175" y="9.3345" size="1.778" layer="27" rot="R270" display="off"/>
-<attribute name="MF" value="" x="3.175" y="9.3345" size="1.778" layer="27" rot="R270" display="off"/>
-<attribute name="OC_FARNELL" value="unknown" x="3.175" y="9.3345" size="1.778" layer="27" rot="R270" display="off"/>
+<element name="X4" library="con-ptr500" package="AK500/2" value="" x="3.175" y="9.525" smashed="yes" rot="R270">
+<attribute name="NAME" x="5.3975" y="9.652" size="1.016" layer="25" ratio="10"/>
+<attribute name="VALUE" x="-2.54" y="14.605" size="1.778" layer="27" ratio="10" rot="R270"/>
+<attribute name="OC_NEWARK" value="unknown" x="3.175" y="9.525" size="1.778" layer="27" rot="R270" display="off"/>
+<attribute name="MPN" value="" x="3.175" y="9.525" size="1.778" layer="27" rot="R270" display="off"/>
+<attribute name="MF" value="" x="3.175" y="9.525" size="1.778" layer="27" rot="R270" display="off"/>
+<attribute name="OC_FARNELL" value="unknown" x="3.175" y="9.525" size="1.778" layer="27" rot="R270" display="off"/>
 </element>
 <element name="IC1" library="uln-udn" package="DIL18" value="ULN2803" x="38.5445" y="24.13" smashed="yes" rot="R270">
@@
 <element name="H1" library="holes" package="3,0" value="MOUNT-HOLE3.0" x="3.6195" y="46.4185" smashed="yes"/>
 <element name="H2" library="holes" package="3,0" value="MOUNT-HOLE3.0" x="21.59" y="4.953" smashed="yes"/>
-<element name="JP1" library="jumper" package="JP2" value="" x="6.35" y="2.54" smashed="yes">
-<attribute name="NAME" x="10.0965" y="3.302" size="1.016" layer="25" ratio="10" rot="R270"/>
-<attribute name="VALUE" x="2.794" y="-0.508" size="1.27" layer="27" ratio="10"/>
-</element>
 <element name="LOGO1" library="SparkFun-Aesthetics" package="OSHW-LOGO-S" value="OSHW-LOGOS" x="4.1275" y="39.497"/>
 <element name="U$2" library="Logo_escorna" package="ESCORNA_PEQUE" value="ESCORNABOT" x="8.3185" y="44.1325"/>
@@
 <element name="U$5" library="escorna" package="ESCORNA_PEQUE" value="ESCORNABOT" x="8.3185" y="44.069"/>
 <element name="U$1" library="escorna" package="ESCORNA_PEQUE" value="ESCORNABOT" x="13.462" y="43.7515" rot="MR0"/>
-<element name="U$6" library="xdesig" package="XDESIG_CU" value="XDESIG" x="8.001" y="44.2595"/>
+<element name="U$6" library="xdesig" package="XDESIG_CU_2" value="XDESIG" x="8.001" y="44.2595"/>
+<element name="S2" library="escorna" package="SK-12F14-G" value="" x="7.3025" y="1.778" smashed="yes">
+<attribute name="VALUE" x="3.3025" y="4.778" size="1.27" layer="27"/>
+<attribute name="NAME" x="10.859" y="2.9045" size="1.27" layer="25"/>
+</element>
 </elements>
 <signals>
@@
 <wire x1="31.75" y1="13.97" x2="31.75" y2="11.43" width="0.8128" layer="16"/>
 <wire x1="24.13" y1="13.97" x2="19.05" y2="13.97" width="0.8128" layer="16"/>
-<wire x1="19.05" y1="13.97" x2="17.78" y2="15.24" width="0.8128" layer="16"/>
-<wire x1="17.78" y1="15.24" x2="15.24" y2="17.78" width="0.8128" layer="16"/>
+<wire x1="19.05" y1="13.97" x2="15.24" y2="17.78" width="0.8128" layer="16"/>
 <wire x1="5.7531" y1="26.0223" x2="5.7531" y2="27.3431" width="0.3048" layer="16"/>
 <wire x1="5.7531" y1="27.3431" x2="6.35" y2="27.94" width="0.3048" layer="16"/>
-<wire x1="15.24" y1="27.94" x2="15.24" y2="17.78" width="0.3048" layer="16"/>
-<wire x1="17.78" y1="15.24" x2="17.78" y2="17.78" width="0.3048" layer="16"/>
+<wire x1="15.24" y1="27.94" x2="15.24" y2="17.907" width="0.3048" layer="16"/>
 <wire x1="17.78" y1="27.94" x2="15.24" y2="30.48" width="0.3048" layer="16"/>
 <contactref element="C1.1" pad="2"/>
@@
 <wire x1="5.1435" y1="19.1135" x2="6.35" y2="20.32" width="0.4064" layer="16"/>
 <wire x1="6.35" y1="20.32" x2="17.78" y2="20.32" width="0.4064" layer="16"/>
-<wire x1="17.78" y1="20.32" x2="17.78" y2="17.78" width="0.4064" layer="16"/>
-<wire x1="17.78" y1="17.78" x2="6.35" y2="17.78" width="0.4064" layer="16"/>
 <wire x1="6.35" y1="17.78" x2="5.08" y2="19.05" width="0.4064" layer="16"/>
 <wire x1="3.81" y1="19.05" x2="5.08" y2="19.05" width="0.4064" layer="16"/>
+<wire x1="6.35" y1="17.78" x2="15.24" y2="17.78" width="0.4064" layer="16"/>
+<wire x1="15.24" y1="17.78" x2="15.24" y2="17.907" width="0.4064" layer="16"/>
+<wire x1="8.89" y1="8.89" x2="6.3246" y2="8.89" width="1.27" layer="16"/>
+<wire x1="6.3246" y1="8.89" x2="3.175" y2="12.0396" width="1.27" layer="16"/>
+<contactref element="S2" pad="P$4"/>
+<contactref element="S2" pad="P$5"/>
 </signal>
 <signal name="RAW">
@@
 <wire x1="49.53" y1="24.13" x2="49.53" y2="10.7315" width="0.8128" layer="16"/>
 <wire x1="49.53" y1="10.7315" x2="49.53" y2="6.731" width="0.8128" layer="16"/>
-<wire x1="49.53" y1="6.731" x2="43.8785" y2="1.0795" width="0.8128" layer="16"/>
-<wire x1="43.8785" y1="1.0795" x2="11.6205" y2="1.0795" width="0.8128" layer="16"/>
-<wire x1="11.6205" y1="1.0795" x2="10.16" y2="2.54" width="0.8128" layer="16"/>
+<wire x1="49.53" y1="6.731" x2="43.7515" y2="0.9525" width="0.8128" layer="16"/>
 <wire x1="49.44" y1="10.6415" x2="49.53" y2="10.7315" width="0.6096" layer="16"/>
 <wire x1="46.7355" y1="10.8955" x2="49.186" y2="10.8955" width="0.8128" layer="16"/>
@@
 <wire x1="15.11" y1="6.35" x2="12.7" y2="6.35" width="0.8128" layer="16"/>
 <wire x1="12.7" y1="6.35" x2="8.89" y2="6.35" width="0.8128" layer="16"/>
-<contactref element="JP1" pad="3"/>
-<wire x1="10.16" y1="2.54" x2="8.89" y2="2.54" width="0.8128" layer="16"/>
-<wire x1="8.89" y1="6.35" x2="8.89" y2="2.54" width="0.8128" layer="16"/>
+<contactref element="S2" pad="P$1"/>
+<contactref element="S2" pad="P$2"/>
+<wire x1="7.3025" y1="1.778" x2="8.89" y2="1.778" width="1.27" layer="16"/>
+<wire x1="8.89" y1="1.778" x2="10.3025" y2="1.778" width="1.27" layer="16"/>
+<wire x1="8.89" y1="6.35" x2="8.89" y2="3.81" width="1.27" layer="16"/>
+<wire x1="8.89" y1="3.81" x2="8.89" y2="1.778" width="1.27" layer="16"/>
+<wire x1="16.383" y1="3.81" x2="8.89" y2="3.81" width="0.8128" layer="16"/>
+<wire x1="16.383" y1="3.81" x2="19.2405" y2="0.9525" width="0.8128" layer="16"/>
+<wire x1="19.2405" y1="0.9525" x2="43.7515" y2="0.9525" width="0.8128" layer="16"/>
 </signal>
 <signal name="D13">
@@
 <contactref element="JP2" pad="2"/>
 <wire x1="47.752" y1="43.688" x2="43.4975" y2="43.688" width="0.8128" layer="16"/>
-</signal>
-<signal name="N$4">
-<contactref element="X4" pad="2"/>
-<wire x1="3.175" y1="6.8199" x2="3.175" y2="4.445" width="1.27" layer="16"/>
-<wire x1="3.175" y1="4.445" x2="3.81" y2="3.81" width="1.27" layer="16"/>
-<contactref element="JP1" pad="1"/>
-<contactref element="JP1" pad="2"/>
-<wire x1="3.81" y1="3.81" x2="3.81" y2="2.54" width="1.27" layer="16"/>
-<wire x1="3.81" y1="2.54" x2="6.35" y2="2.54" width="1.27" layer="16"/>
 </signal>
 <signal name="3V3">
@@
 <wire x1="12.7" y1="13.97" x2="8.89" y2="13.97" width="0.8128" layer="16"/>
 </signal>
+<signal name="N$3">
+<contactref element="X4" pad="2"/>
+<contactref element="S2" pad="P$3"/>
+<wire x1="4.3025" y1="1.778" x2="4.3025" y2="5.8829" width="1.27" layer="16"/>
+<wire x1="4.3025" y1="5.8829" x2="3.175" y2="7.0104" width="1.27" layer="16"/>
+</signal>
 </signals>
