File: Escorna_CPU_1_0/Escorna_CPU_1_01.sch (EAGLE design)
At the start: 25 parts, among them IC1 ULN2803, X3 22-23-2031

Commit message: Xdesig update 2015-06-04
Parts:
- removed JP1: (no value), jumper:JP2E
- added S2: (no value), escorna:SK12F14F
Connections:
- removed net N$4: JP1.1, JP1.2, X4-2.KL
- new net N$3: S2.S, X4-2.KL
- net GND: now also S2.P$1, S2.P$2
- net RAW: now also S2.O, S2.P; no longer JP1.3
Changed lines of the file:
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@@
 <grid distance="0.1" unitdist="inch" unit="inch" style="lines" multiple="1" display="no" altdistance="0.01" altunitdist="inch" altunit="inch"/>
 <layers>
-<layer number="1" name="Top" color="1" fill="1" visible="no" active="no"/>
-<layer number="16" name="Bottom" color="4" fill="1" visible="no" active="no"/>
-<layer number="17" name="Pads" color="2" fill="1" visible="no" active="no"/>
-<layer number="18" name="Vias" color="2" fill="1" visible="no" active="no"/>
-<layer number="19" name="Unrouted" color="6" fill="1" visible="no" active="no"/>
-<layer number="20" name="Dimension" color="15" fill="1" visible="no" active="no"/>
-<layer number="21" name="tPlace" color="7" fill="1" visible="no" active="no"/>
-<layer number="22" name="bPlace" color="7" fill="1" visible="no" active="no"/>
-<layer number="23" name="tOrigins" color="15" fill="1" visible="no" active="no"/>
-<layer number="24" name="bOrigins" color="15" fill="1" visible="no" active="no"/>
-<layer number="25" name="tNames" color="7" fill="1" visible="no" active="no"/>
-<layer number="26" name="bNames" color="7" fill="1" visible="no" active="no"/>
-<layer number="27" name="tValues" color="7" fill="1" visible="no" active="no"/>
-<layer number="28" name="bValues" color="7" fill="1" visible="no" active="no"/>
+<layer number="1" name="Top" color="1" fill="1" visible="yes" active="no"/>
+<layer number="16" name="Bottom" color="4" fill="1" visible="yes" active="no"/>
+<layer number="17" name="Pads" color="2" fill="1" visible="yes" active="no"/>
+<layer number="18" name="Vias" color="2" fill="1" visible="yes" active="no"/>
+<layer number="19" name="Unrouted" color="6" fill="1" visible="yes" active="no"/>
+<layer number="20" name="Dimension" color="15" fill="1" visible="yes" active="no"/>
+<layer number="21" name="tPlace" color="7" fill="1" visible="yes" active="no"/>
+<layer number="22" name="bPlace" color="7" fill="1" visible="yes" active="no"/>
+<layer number="23" name="tOrigins" color="15" fill="1" visible="yes" active="no"/>
+<layer number="24" name="bOrigins" color="15" fill="1" visible="yes" active="no"/>
+<layer number="25" name="tNames" color="7" fill="1" visible="yes" active="no"/>
+<layer number="26" name="bNames" color="7" fill="1" visible="yes" active="no"/>
+<layer number="27" name="tValues" color="7" fill="1" visible="yes" active="no"/>
+<layer number="28" name="bValues" color="7" fill="1" visible="yes" active="no"/>
 <layer number="29" name="tStop" color="7" fill="3" visible="no" active="no"/>
 <layer number="30" name="bStop" color="7" fill="6" visible="no" active="no"/>
@@
 <layer number="35" name="tGlue" color="7" fill="4" visible="no" active="no"/>
 <layer number="36" name="bGlue" color="7" fill="5" visible="no" active="no"/>
-<layer number="37" name="tTest" color="7" fill="1" visible="no" active="no"/>
-<layer number="38" name="bTest" color="7" fill="1" visible="no" active="no"/>
+<layer number="37" name="tTest" color="7" fill="1" visible="yes" active="no"/>
+<layer number="38" name="bTest" color="7" fill="1" visible="yes" active="no"/>
 <layer number="39" name="tKeepout" color="4" fill="11" visible="no" active="no"/>
 <layer number="40" name="bKeepout" color="1" fill="11" visible="no" active="no"/>
@@
 <layer number="44" name="Drills" color="7" fill="1" visible="no" active="no"/>
 <layer number="45" name="Holes" color="7" fill="1" visible="no" active="no"/>
-<layer number="46" name="Milling" color="3" fill="1" visible="no" active="no"/>
-<layer number="47" name="Measures" color="7" fill="1" visible="no" active="no"/>
-<layer number="48" name="Document" color="7" fill="1" visible="no" active="no"/>
-<layer number="49" name="Reference" color="7" fill="1" visible="no" active="no"/>
-<layer number="50" name="dxf" color="7" fill="1" visible="no" active="no"/>
-<layer number="51" name="tDocu" color="7" fill="1" visible="no" active="no"/>
-<layer number="52" name="bDocu" color="7" fill="1" visible="no" active="no"/>
-<layer number="53" name="tGND_GNDA" color="7" fill="9" visible="no" active="no"/>
-<layer number="54" name="bGND_GNDA" color="1" fill="9" visible="no" active="no"/>
-<layer number="56" name="wert" color="7" fill="1" visible="no" active="no"/>
-<layer number="57" name="tCAD" color="7" fill="1" visible="no" active="no"/>
+<layer number="46" name="Milling" color="3" fill="1" visible="yes" active="no"/>
+<layer number="47" name="Measures" color="7" fill="1" visible="yes" active="no"/>
+<layer number="48" name="Document" color="7" fill="1" visible="yes" active="no"/>
+<layer number="49" name="Reference" color="7" fill="1" visible="yes" active="no"/>
+<layer number="50" name="dxf" color="7" fill="1" visible="yes" active="no"/>
+<layer number="51" name="tDocu" color="7" fill="1" visible="yes" active="no"/>
+<layer number="52" name="bDocu" color="7" fill="1" visible="yes" active="no"/>
+<layer number="53" name="tGND_GNDA" color="7" fill="9" visible="yes" active="no"/>
+<layer number="54" name="bGND_GNDA" color="1" fill="9" visible="yes" active="no"/>
+<layer number="56" name="wert" color="7" fill="1" visible="yes" active="no"/>
+<layer number="57" name="tCAD" color="7" fill="1" visible="yes" active="no"/>
 <layer number="91" name="Nets" color="2" fill="1" visible="yes" active="yes"/>
 <layer number="92" name="Busses" color="1" fill="1" visible="yes" active="yes"/>
@@
 <part name="H1" library="holes" deviceset="MOUNT-HOLE" device="3.0"/>
 <part name="H2" library="holes" deviceset="MOUNT-HOLE" device="3.0"/>
-<part name="JP1" library="jumper" deviceset="JP2E" device=""/>
 <part name="LOGO1" library="SparkFun-Aesthetics" deviceset="OSHW-LOGO" device="S"/>
 <part name="U$6" library="xdesig" deviceset="XDESIG" device=""/>
 <part name="U$1" library="escorna" deviceset="ESCORNABOT" device=""/>
+<part name="S2" library="escorna" deviceset="SK12F14" device="F"/>
 </parts>
 <sheets>
@@
 <instance part="H1" gate="G$1" x="93.98" y="22.86"/>
 <instance part="H2" gate="G$1" x="93.98" y="30.48"/>
-<instance part="JP1" gate="1" x="40.64" y="25.4"/>
 <instance part="LOGO1" gate="G$1" x="248.92" y="48.26"/>
 <instance part="U$6" gate="G$1" x="259.08" y="17.78"/>
 <instance part="U$1" gate="G$1" x="7.62" y="160.02"/>
+<instance part="S2" gate="S$" x="44.196" y="22.86" rot="MR0"/>
 </instances>
 <busses>
@@
 <junction x="63.5" y="10.16"/>
 <pinref part="C1.1" gate="G$1" pin="2"/>
+<pinref part="S2" gate="S$" pin="P$1"/>
+<wire x1="50.546" y1="15.24" x2="52.07" y2="15.24" width="0.1524" layer="91"/>
+<wire x1="52.07" y1="15.24" x2="52.07" y2="10.16" width="0.1524" layer="91"/>
+<wire x1="52.07" y1="10.16" x2="52.07" y2="9.906" width="0.1524" layer="91"/>
+<wire x1="63.5" y1="10.16" x2="52.07" y2="10.16" width="0.1524" layer="91"/>
+<junction x="52.07" y="10.16"/>
 </segment>
 <segment>
@@
 <wire x1="17.78" y1="12.7" x2="17.78" y2="10.16" width="0.1524" layer="91"/>
 <pinref part="SUPPLY6" gate="GND" pin="GND"/>
+<wire x1="17.78" y1="12.7" x2="33.02" y2="12.7" width="0.1524" layer="91"/>
+<wire x1="33.02" y1="12.7" x2="33.02" y2="15.24" width="0.1524" layer="91"/>
+<junction x="17.78" y="12.7"/>
+<pinref part="S2" gate="S$" pin="P$2"/>
+<wire x1="33.02" y1="15.24" x2="37.846" y2="15.24" width="0.1524" layer="91"/>
 </segment>
 <segment>
@@
 <segment>
 <pinref part="C1" gate="G$1" pin="1"/>
-<wire x1="43.18" y1="22.86" x2="63.5" y2="22.86" width="0.1524" layer="91"/>
-<label x="50.8" y="25.4" size="2.54" layer="95"/>
+<label x="63.5" y="25.4" size="2.54" layer="95"/>
 <wire x1="73.66" y1="22.86" x2="63.5" y2="22.86" width="0.1524" layer="91"/>
+<pinref part="C1.1" gate="G$1" pin="1"/>
+<wire x1="50.546" y1="22.86" x2="63.5" y2="22.86" width="0.1524" layer="91"/>
 <junction x="63.5" y="22.86"/>
-<pinref part="C1.1" gate="G$1" pin="1"/>
-<pinref part="JP1" gate="1" pin="3"/>
+<pinref part="S2" gate="S$" pin="P"/>
 </segment>
 <segment>
@@
 <wire x1="50.8" y1="86.36" x2="43.18" y2="86.36" width="0.1524" layer="91"/>
 <label x="43.18" y="86.36" size="1.778" layer="95"/>
+</segment>
+<segment>
+<pinref part="S2" gate="S$" pin="O"/>
+<wire x1="37.846" y1="25.4" x2="33.528" y2="25.4" width="0.1524" layer="91"/>
+<label x="33.02" y="25.4" size="1.778" layer="95"/>
 </segment>
 </net>
@@
 <wire x1="114.3" y1="71.12" x2="99.06" y2="71.12" width="0.1524" layer="91"/>
 <pinref part="JP2" gate="1" pin="2"/>
-</segment>
-</net>
-<net name="N$4" class="0">
-<segment>
-<pinref part="X4" gate="-2" pin="KL"/>
-<wire x1="40.64" y1="22.86" x2="38.1" y2="22.86" width="0.1524" layer="91"/>
-<label x="20.32" y="25.4" size="1.778" layer="95"/>
-<pinref part="JP1" gate="1" pin="1"/>
-<wire x1="38.1" y1="22.86" x2="17.78" y2="22.86" width="0.1524" layer="91"/>
-<junction x="38.1" y="22.86"/>
-<pinref part="JP1" gate="1" pin="2"/>
 </segment>
 </net>
@@
 </segment>
 </net>
+<net name="N$3" class="0">
+<segment>
+<pinref part="X4" gate="-2" pin="KL"/>
+<wire x1="30.734" y1="22.86" x2="17.78" y2="22.86" width="0.1524" layer="91"/>
+<pinref part="S2" gate="S$" pin="S"/>
+<wire x1="30.734" y1="20.32" x2="30.734" y2="22.86" width="0.1524" layer="91"/>
+<wire x1="37.846" y1="20.32" x2="30.734" y2="20.32" width="0.1524" layer="91"/>
+</segment>
+</net>
