File: Cervus_1_0/Cervus_1_0.brd (EAGLE design)
At the start: 50.5 x 50.8 mm, 52 parts, among them IC1 NCP1117ST50T3G, IC2 ULN2803, Q1 SPK-5032 16MHz, U1 ATMEGA32U4-XUAU, U2 MICRO USB, U3 LP2985-33DBVR, X2 AK550/2

Commit message: Actualización nome
comprobado e funcional
Parts:
- moved X2 0.58 mm to (21.4, 2.02)
Changed lines of the file:
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@@
 <setting verticaltext="up"/>
 </settings>
-<grid distance="0.05" unitdist="inch" unit="mm" style="lines" multiple="1" display="no" altdistance="0.065" altunitdist="mm" altunit="mm"/>
+<grid distance="0.05" unitdist="inch" unit="mil" style="lines" multiple="1" display="no" altdistance="2.55905512" altunitdist="mil" altunit="mil"/>
 <layers>
-<layer number="1" name="Top" color="4" fill="1" visible="no" active="yes"/>
-<layer number="16" name="Bottom" color="1" fill="1" visible="no" active="yes"/>
+<layer number="1" name="Top" color="4" fill="1" visible="yes" active="yes"/>
+<layer number="16" name="Bottom" color="1" fill="1" visible="yes" active="yes"/>
 <layer number="17" name="Pads" color="2" fill="1" visible="yes" active="yes"/>
-<layer number="18" name="Vias" color="2" fill="1" visible="no" active="yes"/>
+<layer number="18" name="Vias" color="6" fill="1" visible="yes" active="yes"/>
 <layer number="19" name="Unrouted" color="6" fill="1" visible="no" active="yes"/>
 <layer number="20" name="Dimension" color="15" fill="1" visible="yes" active="yes"/>
-<layer number="21" name="tPlace" color="7" fill="1" visible="yes" active="yes"/>
+<layer number="21" name="tPlace" color="7" fill="1" visible="no" active="yes"/>
 <layer number="22" name="bPlace" color="7" fill="1" visible="no" active="yes"/>
 <layer number="23" name="tOrigins" color="15" fill="1" visible="no" active="yes"/>
 <layer number="24" name="bOrigins" color="15" fill="1" visible="no" active="yes"/>
-<layer number="25" name="tNames" color="7" fill="1" visible="yes" active="yes"/>
+<layer number="25" name="tNames" color="7" fill="1" visible="no" active="yes"/>
 <layer number="26" name="bNames" color="7" fill="1" visible="no" active="yes"/>
 <layer number="27" name="tValues" color="7" fill="1" visible="no" active="yes"/>
@@
 <layer number="49" name="Reference" color="7" fill="1" visible="no" active="yes"/>
 <layer number="50" name="dxf" color="7" fill="1" visible="no" active="no"/>
-<layer number="51" name="tDocu" color="7" fill="1" visible="yes" active="yes"/>
+<layer number="51" name="tDocu" color="7" fill="1" visible="no" active="yes"/>
 <layer number="52" name="bDocu" color="7" fill="1" visible="no" active="yes"/>
 <layer number="53" name="tGND_GNDA" color="7" fill="9" visible="no" active="no"/>
@@
 </class>
 </classes>
-<designrules name="default">
+<designrules name="default *">
 <description language="de">&lt;b&gt;EAGLE Design Rules&lt;/b&gt;
 &lt;p&gt;
@@
 <param name="mtCopper" value="0.035mm 0.035mm 0.035mm 0.035mm 0.035mm 0.035mm 0.035mm 0.035mm 0.035mm 0.035mm 0.035mm 0.035mm 0.035mm 0.035mm 0.035mm 0.035mm"/>
 <param name="mtIsolate" value="1.5mm 0.15mm 0.2mm 0.15mm 0.2mm 0.15mm 0.2mm 0.15mm 0.2mm 0.15mm 0.2mm 0.15mm 0.2mm 0.15mm 0.2mm"/>
-<param name="mdWireWire" value="8mil"/>
-<param name="mdWirePad" value="8mil"/>
-<param name="mdWireVia" value="8mil"/>
+<param name="mdWireWire" value="10mil"/>
+<param name="mdWirePad" value="10mil"/>
+<param name="mdWireVia" value="10mil"/>
 <param name="mdPadPad" value="8mil"/>
-<param name="mdPadVia" value="8mil"/>
-<param name="mdViaVia" value="8mil"/>
+<param name="mdPadVia" value="12mil"/>
+<param name="mdViaVia" value="12mil"/>
 <param name="mdSmdPad" value="8mil"/>
 <param name="mdSmdVia" value="8mil"/>
@@
 <param name="mdViaViaSameLayer" value="8mil"/>
 <param name="mnLayersViaInSmd" value="2"/>
-<param name="mdCopperDimension" value="40mil"/>
-<param name="mdDrill" value="8mil"/>
+<param name="mdCopperDimension" value="24mil"/>
+<param name="mdDrill" value="12mil"/>
 <param name="mdSmdStop" value="0mil"/>
 <param name="msWidth" value="10mil"/>
-<param name="msDrill" value="24mil"/>
+<param name="msDrill" value="22mil"/>
 <param name="msMicroVia" value="9.99mm"/>
 <param name="msBlindViaRatio" value="0.5"/>
@@
 <param name="rlMinPadBottom" value="10mil"/>
 <param name="rlMaxPadBottom" value="20mil"/>
-<param name="rlMinViaOuter" value="8mil"/>
+<param name="rlMinViaOuter" value="10mil"/>
 <param name="rlMaxViaOuter" value="20mil"/>
 <param name="rlMinViaInner" value="8mil"/>
@@
 <param name="psBottom" value="-1"/>
 <param name="psFirst" value="-1"/>
-<param name="psElongationLong" value="100"/>
+<param name="psElongationLong" value="50"/>
 <param name="psElongationOffset" value="100"/>
-<param name="mvStopFrame" value="1"/>
-<param name="mvCreamFrame" value="0"/>
-<param name="mlMinStopFrame" value="4mil"/>
+<param name="mvStopFrame" value="0.05"/>
+<param name="mvCreamFrame" value="0.1"/>
+<param name="mlMinStopFrame" value="2mil"/>
 <param name="mlMaxStopFrame" value="4mil"/>
-<param name="mlMinCreamFrame" value="0mil"/>
-<param name="mlMaxCreamFrame" value="0mil"/>
-<param name="mlViaStopLimit" value="0mil"/>
-<param name="srRoundness" value="0"/>
-<param name="srMinRoundness" value="0mil"/>
-<param name="srMaxRoundness" value="0mil"/>
+<param name="mlMinCreamFrame" value="2mil"/>
+<param name="mlMaxCreamFrame" value="20mil"/>
+<param name="mlViaStopLimit" value="30mil"/>
+<param name="srRoundness" value="1"/>
+<param name="srMinRoundness" value="2mil"/>
+<param name="srMaxRoundness" value="10mil"/>
 <param name="slThermalIsolate" value="10mil"/>
 <param name="slThermalsForVias" value="0"/>
@@
 <element name="U3" library="SmartPrj" package="SOT23-DBV" value="LP2985-33DBVR" x="17.43" y="9.22" smashed="yes" rot="R270">
 <attribute name="NAME" x="17.845" y="8.7" size="0.6096" layer="25" rot="R90"/>
-<attribute name="VALUE" x="14.001" y="11.125" size="1.27" layer="27" rot="R270"/>
+<attribute name="VALUE" x="17.724" y="10.77" size="0.5" layer="27" rot="R90"/>
 </element>
 <element name="SV1" library="con-lsta" package="FE15" value="SH-BI-196*15" x="2.54" y="24.13" smashed="yes" rot="R270">
@@
 <attribute name="VALUE" x="37.542" y="-2.909" size="1.27" layer="27" ratio="10"/>
 </element>
-<element name="X2" library="con-ptr500" package="AK550/2" value="AK550/2" x="21.42" y="2.605" smashed="yes">
-<attribute name="OC_NEWARK" value="unknown" x="21.42" y="2.605" size="1.778" layer="27" display="off"/>
-<attribute name="MPN" value="" x="21.42" y="2.605" size="1.778" layer="27" display="off"/>
-<attribute name="MF" value="" x="21.42" y="2.605" size="1.778" layer="27" display="off"/>
-<attribute name="OC_FARNELL" value="unknown" x="21.42" y="2.605" size="1.778" layer="27" display="off"/>
-<attribute name="NAME" x="21.075" y="3.455" size="0.6096" layer="25"/>
-<attribute name="VALUE" x="18.245" y="-3.11" size="1.778" layer="27"/>
+<element name="X2" library="con-ptr500" package="AK550/2" value="AK550/2" x="21.42" y="2.02" smashed="yes">
+<attribute name="OC_NEWARK" value="unknown" x="21.42" y="2.02" size="1.778" layer="27" display="off"/>
+<attribute name="MPN" value="" x="21.42" y="2.02" size="1.778" layer="27" display="off"/>
+<attribute name="MF" value="" x="21.42" y="2.02" size="1.778" layer="27" display="off"/>
+<attribute name="OC_FARNELL" value="unknown" x="21.42" y="2.02" size="1.778" layer="27" display="off"/>
+<attribute name="NAME" x="21.075" y="2.87" size="0.6096" layer="25"/>
+<attribute name="VALUE" x="18.245" y="-3.695" size="1.778" layer="27"/>
 </element>
 <element name="C11" library="SmartPrj" package="C0603-ROUND" value="22p" x="29.96" y="31.17" smashed="yes" rot="R90">
@@
 </element>
 <element name="LOGO1" library="SparkFun-Aesthetics" package="OSHW-LOGO-S" value="OSHW-LOGOS" x="34.86" y="29.41"/>
-<element name="S1" library="escorna" package="SK-12D07" value="SK-12D07" x="10.39" y="2.54"/>
+<element name="S1" library="escorna" package="SK-12D07" value="SK-12D07" x="10.39" y="2.54" smashed="yes">
+<attribute name="VALUE" x="6.39" y="5.54" size="1.27" layer="27"/>
+<attribute name="NAME" x="6.39" y="7.54" size="1.27" layer="25"/>
+</element>
 <element name="U$5" library="xdesig" package="XDESIG" value="XDESIG21" x="17.315" y="4.005" rot="MR0"/>
 <element name="JP2" library="jumper" package="JP1" value="" x="12.515" y="27.515"/>
-<element name="D1" library="diode" package="SMA" value="" x="10.6" y="9.055"/>
+<element name="D1" library="diode" package="SMA" value="" x="10.6" y="9.055" smashed="yes">
+<attribute name="NAME" x="7.85" y="11.055" size="1.27" layer="25" ratio="10"/>
+<attribute name="VALUE" x="7.85" y="5.555" size="1.27" layer="27" ratio="10"/>
+</element>
 <element name="U$6" library="escorna" package="ESCORNA_QR25" value="QR25" x="25.785" y="23.97" rot="MR0"/>
 <element name="U$3" library="escorna" package="ESCORNA_PEQUE" value="ESCORNABOT" x="34.86" y="15.85"/>
@@
 <via x="4.645" y="27.8964" extent="1-16" drill="0.6096" diameter="0.8596"/>
 <via x="4.645" y="25.3614" extent="1-16" drill="0.6096" diameter="0.8596"/>
+<wire x1="26.25" y1="32.065" x2="28.45" y2="30.465" width="0" layer="19" extent="1-1"/>
 </signal>
 <signal name="UVCC">
@@
 <contactref element="X2" pad="1"/>
 <contactref element="S1" pad="P$2"/>
-<wire x1="19.67" y1="2.605" x2="18.985" y2="2.605" width="1.016" layer="1"/>
+<wire x1="19.67" y1="2.02" x2="18.985" y2="2.605" width="1.016" layer="1"/>
 <wire x1="18.985" y1="2.605" x2="16.51" y2="5.08" width="1.016" layer="1"/>
 <wire x1="16.51" y1="5.08" x2="13.97" y2="5.08" width="1.016" layer="1"/>
