File: EscornaCPU/1.20/Escorna_CPU_1_20.sch (EAGLE design)
At the start: 88 parts, among them IC1 ULN2803, J1 2.54, U2 ESP01, U6 1117-3.3, X1 AK550/2, X1.1 AK550/2

Commit message: New design
Parts:
- removed C1.2: 1uF, rcl:C-EUC1206
- removed C2.1: 100nF, rcl:C-EUC1206
- removed D2: K7, adafruit:DIODESMA
- removed ESC: ESCORNABOT, escorna:ESCORNABOT
- removed H1, H2: MOUNT-HOLE3.0, holes:MOUNT-HOLE3.0
- removed J1: 2.54, con-molex:22-27-2021-02
- removed LED1, LED2, LED3, LED4: (no value), adafruit:LED3MM
- removed LED1.1, LED2.1, LED3.1, LED4.1: (no value), adafruit:LEDCHIPLED_0603
- removed R10, R6, R8, R9: 1K, rcl:R-EU_0204/7
- removed R10.1, R6.1, R8.1, R9.1: 1K, rcl:R-EU_R0603
- removed R11, R12, R14, R7: 10K, rcl:R-EU_0204/7
- removed R11.1, R12.1, R14.1, R7.1: 10K, rcl:R-EU_R0603
- removed R13: 18K, rcl:R-EU_0204/7
- removed R13.1: 18K, rcl:R-EU_R0603
- removed S1, S2, S3, S4, S5: (no value), switch-omron:10-XX
- removed S1.1, S2.1, S3.1, S4.1, S5.1: (no value), switch-omron:40-XX
- removed SG1: F/CM12P, buzzer:F/CM12P
- removed SJ2: (no value), jumper:SJ
- removed U$11, U$3, U$6: FRECHA, escorna:FRECHA
- removed U$2: GO, escorna:GO
- added C3: 100nF, rcl:C-EU025-025X050
- added C3.1: 100nF, rcl:C-EUC0603K
- added D1.1: M7, diode:SCHOTTKY-DIODE
- added ESC1, ESC2: ESCORNABOT, escorna:ESCORNABOT
- added JP2: (no value), SparkFunEagle-6-6-07:JP1E
- added JP3, JP4: (no value), jumper:JP1E
- added JP5: (no value), jumper:JP4E
- added LOGO2: OSHW-LOGOS, SparkFun-Aesthetics:OSHW-LOGOS
- added SV5, SV6: (no value), con-lstb:MA06-1
- added Z1: CFG12, buzzer:F/CM12P
- C1.1: device rcl:C-EUC1206 -> rcl:C-EUC0603K
- C2: value 100nF -> 1uF; device rcl:C-EU025-025X050 -> rcl:C-EUC1206K
- H3, H4: value MOUNT-HOLE3.0 -> H3.0
- JP1: device jumper:JP1E -> SparkFunEagle-6-6-07:JP1E
- R3, R3.1: value 10K -> 18K
- R5, R5.1: value 22K -> 10K
- SV1: value (none) -> 1x15 SOCKET STRIP; device con-lstb:MA08-2 -> escorna_LBREscorna_CPU_2_10:CON-LSTA_FE15-1
- SV2: value (none) -> 1x15 SOCKET STRIP
- SV3: device escorna_LBREscorna_CPU_2_10:CON-LSTA_FE15-1 -> con-lstb:MA06-1
- SV4: device con-lstb:MA04-1 -> con-lstb:MA06-1
- U$1: value FRECHA -> XDESIG_XDESIG21; device escorna:FRECHA -> Escorna_CPU_2_01:XDESIG_XDESIG21
Connections:
- removed net K: LED1.1.C, LED1.C, LED2.1.C, LED2.C, LED3.1.C, LED3.C, LED4.1.C, LED4.C, SJ2.2
- removed net N$12: F1.1, F1.1.1, J1-1.S, X1-1.KL, X1.1-1.KL
- removed net N$14: R14.1, R14.1.1, U2.GPIO0
- removed net N$4: LED2.1.A, LED2.A, R8.1.2, R8.2
- removed net N$5: LED1.1.A, LED1.A, R6.1.2, R6.2
- removed net N$6: LED3.1.A, LED3.A, R9.1.2, R9.2
- removed net N$8: LED4.1.A, LED4.A, R10.1, R10.1.2
- removed net S1: R1.1, R1.1.1, R2.1.2, R2.2, S1.1.P, S1.1.P1, S1.P, S1.P1
- removed net S2: R2.1, R2.1.1, R3.1.2, R3.2, S2.1.P, S2.1.P1, S2.P, S2.P1
- removed net S3: R3.1, R3.1.1, R4.1.2, R4.2, S3.1.P, S3.1.P1, S3.P, S3.P1
- removed net S4: R5.1, R5.1.1, S4.1.P, S4.1.P1, S4.P, S4.P1
- removed net S5: R4.1, R4.1.1, R5.1.2, R5.2, S5.1.P, S5.1.P1, S5.P, S5.P1
- new net N$1: R5.1.2, R5.2, U2.CH_PD
- new net VIN: D1.1.C, D1.C, F1.1.2, F1.2, S7.1.P, S7.1.S, S7.P, S7.S
- net 3V3: now also R4.1, R4.1.1, R5.1, R5.1.1; no longer R11.1, R11.1.1, R14.1.2, R14.2, SV1.15, SV1.16
- net 5V: now also JP3.1, JP3.2, JP5.3, R1.1, R1.1.1, SV4.1, SV4.2, SV4.4, SV4.5, SV4.6; no longer R7.1, R7.1.1, SV1.11, SV1.12
- net A0: now also SV6.1; no longer R6.1, R6.1.1, SV1.9
- net A1: now also SV6.2; no longer R8.1, R8.1.1, SV1.8
- net A2: now also SV6.3; no longer R9.1, R9.1.1, SV1.7
- net A3: now also SV6.4; no longer R10.1.1, R10.2, SV1.6
- net A4: now also JP5.1, SV3.1; no longer SV1.5, SV4.1
- net A5: now also JP5.2, SV3.2; no longer SV1.4, SV4.2
- net A6: now also SV3.3; no longer SV1.3
- net A7: now also SV6.5; no longer R7.1.2, R7.2
- net CH: now also R4.1.2, R4.2, U2.GPIO0; no longer R11.1.2, R11.2, U2.CH_PD
- net D10: now also SV1.13; no longer SV3.13
- net D11: now also SV1.14, SV3.4; no longer SV1.13, SV3.14
- net D12: now also SV1.15, SV3.5; no longer SV1.14, SV3.15
- net D13: now also SV3.6; no longer SV1.10
- net D2: now also SV1.5; no longer SV3.5
- net D3: now also SV1.6; no longer SV3.6
- net D4: now also SV1.7; no longer SV3.7
- net D5: now also SV1.8; no longer SV3.8
- net D6: now also SV1.9; no longer SV3.9
- net D7: now also SV1.10; no longer SV3.10
- net D8: now also SV1.11; no longer SV3.11
- net D9: now also SV1.12; no longer SV3.12
- net GND: now also C1.2, C3.1, C3.1.1, D1.1.A, JP2.1, JP4.1, JP4.2, JP5.4, R3.1.1, R3.2, SV1.4, SV5.1, SV5.2, SV5.3, SV5.4, SV5.5, SV5.6, SV6.6, X1-1.KL, Z1.2; no longer C1.1, C1.2.1, C2.1.1, D2.A, J1-2.S, R13.1.1, R13.2, S1.1.S, S1.1.S1, S1.S, S1.S1, S2.1.S, S2.1.S1, S2.S, S2.S1, S3.1.S, S3.1.S1, S3.S, S3.S1, S4.1.S, S4.1.S1, S4.S, S4.S1, S5.1.S, S5.1.S1, S5.S, S5.S1, SG1.2, SJ2.1, SV1.1, SV1.2, SV3.4, SV4.4, X1-2.KL
- net N$2: now also Z1.1; no longer SG1.1
- net N$3: now also F1.1, F1.1.1, JP2.2, X1-2.KL, X1.1-1.KL; no longer D1.C, D2.C, F1.1.2, F1.2, S7.1.O, S7.O
- net RAW: now also C1.1, C3.1.2, C3.2, S7.1.O, S7.O; no longer C1.2, C1.2.2, C2.1.2, S7.1.P, S7.1.S, S7.P, S7.S
- net RX: now also SV1.2; no longer SV3.2
- net TX: now also R2.1, R2.1.1, SV1.1; no longer R12.1, R12.1.1, SV3.1
- net TX3V3: now also R2.1.2, R2.2, R3.1, R3.1.2; no longer R12.1.2, R12.2, R13.1, R13.1.2
Other:
- note added: "Buzz on"
- note added: "By XDeSIG"
- note added: "Connector to keypad leds.."
- note added: "to Servos, sensors..."
- note added: "to oled I2C..."
- note removed: "Backward"
- note removed: "Choose one Dx.1 = SMD Dx = THT"
- note removed: "D10 ( NANO )"
- note removed: "Enabling LEDs, Default on"
- note removed: "Escornabot Singularis by XDeSIG"
- note removed: "Forward"
- note removed: "Go"
- note removed: "KEYPAD"
- note removed: "Left"
- note removed: "Right"
- note removed: "S1"
- note removed: "S2"
- note removed: "S3"
- note removed: "S4"
- note removed: "S5"
- note removed: "SX SW 6mm"
- note removed: "SX.1 SW12mm"
- note removed: "choose arduino board or jumper out to mute"
- moved on the sheet: C1, C1.1, C2, D1, F1, F1.1, H3, H4, IC1, JP1, R1, R1.1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
