File: EscornaCPU/2.x/2.12/Escorna_CPU_2_12.brd (EAGLE design)
At the start: 49.9 x 89.6 mm, 97 parts, among them IC1 ULN2803, J1 2.54, U2 ESP01, U6 1117-3.3, X1 AK550/2, X1.1 AK550/2

Commit message: New docus
Routing:
- net N$3: track 39.4 -> 40.6 mm, vias 0 -> 1
Changed lines of the file:
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@@
 <grid distance="0.5" unitdist="mm" unit="mm" style="lines" multiple="1" display="no" altdistance="0.05" altunitdist="mm" altunit="mm"/>
 <layers>
-<layer number="1" name="Top" color="1" fill="1" visible="no" active="yes"/>
+<layer number="1" name="Top" color="1" fill="1" visible="yes" active="yes"/>
 <layer number="2" name="Route2" color="1" fill="3" visible="no" active="no"/>
 <layer number="3" name="Route3" color="4" fill="3" visible="no" active="no"/>
@@
 <layer number="14" name="Route14" color="1" fill="6" visible="no" active="no"/>
 <layer number="15" name="Route15" color="4" fill="6" visible="no" active="no"/>
-<layer number="16" name="Bottom" color="4" fill="1" visible="no" active="yes"/>
+<layer number="16" name="Bottom" color="4" fill="1" visible="yes" active="yes"/>
 <layer number="17" name="Pads" color="2" fill="1" visible="yes" active="yes"/>
 <layer number="18" name="Vias" color="2" fill="1" visible="yes" active="yes"/>
-<layer number="19" name="Unrouted" color="6" fill="1" visible="no" active="yes"/>
+<layer number="19" name="Unrouted" color="6" fill="1" visible="yes" active="yes"/>
 <layer number="20" name="Dimension" color="15" fill="1" visible="yes" active="yes"/>
-<layer number="21" name="tPlace" color="7" fill="1" visible="yes" active="yes"/>
+<layer number="21" name="tPlace" color="7" fill="1" visible="no" active="yes"/>
 <layer number="22" name="bPlace" color="7" fill="1" visible="no" active="yes"/>
-<layer number="23" name="tOrigins" color="15" fill="1" visible="yes" active="yes"/>
+<layer number="23" name="tOrigins" color="15" fill="1" visible="no" active="yes"/>
 <layer number="24" name="bOrigins" color="15" fill="1" visible="no" active="yes"/>
-<layer number="25" name="tNames" color="7" fill="1" visible="yes" active="yes"/>
+<layer number="25" name="tNames" color="7" fill="1" visible="no" active="yes"/>
 <layer number="26" name="bNames" color="7" fill="1" visible="no" active="yes"/>
-<layer number="27" name="tValues" color="7" fill="1" visible="yes" active="yes"/>
+<layer number="27" name="tValues" color="7" fill="1" visible="no" active="yes"/>
 <layer number="28" name="bValues" color="7" fill="1" visible="no" active="yes"/>
 <layer number="29" name="tStop" color="7" fill="3" visible="no" active="yes"/>
@@
 <layer number="45" name="Holes" color="7" fill="1" visible="no" active="yes"/>
 <layer number="46" name="Milling" color="3" fill="1" visible="no" active="yes"/>
-<layer number="47" name="Measures" color="7" fill="1" visible="yes" active="yes"/>
+<layer number="47" name="Measures" color="7" fill="1" visible="no" active="yes"/>
 <layer number="48" name="Document" color="7" fill="1" visible="no" active="yes"/>
 <layer number="49" name="Reference" color="7" fill="1" visible="no" active="yes"/>
@@
 <wire x1="45.593" y1="4.593" x2="49" y2="8" width="1.27" layer="16"/>
 <wire x1="49" y1="8" x2="49" y2="31.41" width="1.27" layer="16"/>
-<wire x1="48.2" y1="34.9505" x2="44.6405" y2="34.9505" width="1.27" layer="1"/>
 <wire x1="44.6405" y1="34.9505" x2="44.55" y2="34.86" width="1.27" layer="1"/>
 <wire x1="44.55" y1="34.86" x2="44.55" y2="35.968" width="1.27" layer="1"/>
 <wire x1="44.55" y1="35.968" x2="44.57" y2="35.988" width="1.27" layer="1"/>
 <wire x1="49" y1="31.41" x2="48.2" y2="32.21" width="1.27" layer="16"/>
+<via x="44.6405" y="34.9505" extent="1-16" drill="0.6" shape="square"/>
+<wire x1="44.6405" y1="34.9505" x2="45.4595" y2="34.9505" width="1.27" layer="16"/>
+<wire x1="45.4595" y1="34.9505" x2="48.2" y2="32.21" width="1.27" layer="16"/>
 </signal>
 <signal name="S3">
