File: EscornaCPU/2.x/2.20/Escorna_CPU_2_20.brd (EAGLE design)
At the start: 50 x 100.1 mm, 105 parts, among them IC1 ULN2803, U2 ESP01, U6 ASM1117-3.3, X1 AK550/2, X1.1 AK550/2

Commit message: Upgrade
cambios en 2.20
Parts:
- LED3.1: value Orange -> Orang
Other:
- outline, holes or cut-outs redrawn

Commit message: Upgrade
Resolve bug
Connections:
- net CH: no longer U2.GPIO0
Routing:
- net CH: track 16.4 -> 15.3 mm
Changed lines of the file:
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@@
 <grid distance="0.5" unitdist="mm" unit="mm" style="lines" multiple="1" display="no" altdistance="0.05" altunitdist="mm" altunit="mm"/>
 <layers>
-<layer number="1" name="Top" color="4" fill="1" visible="no" active="yes"/>
+<layer number="1" name="Top" color="4" fill="1" visible="yes" active="yes"/>
 <layer number="2" name="Route2" color="1" fill="3" visible="no" active="no"/>
 <layer number="3" name="Route3" color="4" fill="3" visible="no" active="no"/>
@@
 <layer number="14" name="Route14" color="1" fill="6" visible="no" active="no"/>
 <layer number="15" name="Route15" color="4" fill="6" visible="no" active="no"/>
-<layer number="16" name="Bottom" color="1" fill="1" visible="no" active="yes"/>
+<layer number="16" name="Bottom" color="1" fill="1" visible="yes" active="yes"/>
 <layer number="17" name="Pads" color="2" fill="1" visible="yes" active="yes"/>
 <layer number="18" name="Vias" color="2" fill="1" visible="yes" active="yes"/>
@@
 </signal>
 <signal name="CH">
-<contactref element="U2" pad="CH_PD"/>
-<contactref element="U2" pad="GPIO0"/>
 <contactref element="R13" pad="2"/>
-<wire x1="43.467" y1="87.4595" x2="40.927" y2="84.9195" width="0.4064" layer="16"/>
 <wire x1="48.76" y1="79.2" x2="48.76" y2="81.5" width="0.4064" layer="1"/>
 <wire x1="48.76" y1="81.5" x2="48.76" y2="84.24" width="0.4064" layer="1"/>
 <wire x1="48.76" y1="84.24" x2="46.95" y2="86.05" width="0.4064" layer="1"/>
-<wire x1="46.95" y1="86.05" x2="44.8765" y2="86.05" width="0.4064" layer="1"/>
-<wire x1="44.8765" y1="86.05" x2="43.467" y2="87.4595" width="0.4064" layer="1"/>
 <contactref element="R13.1" pad="2"/>
 <wire x1="47.7" y1="81.2" x2="48.46" y2="81.2" width="0.4064" layer="1"/>
 <wire x1="48.46" y1="81.2" x2="48.76" y2="81.5" width="0.4064" layer="1"/>
+<contactref element="U2" pad="CH_PD"/>
+<wire x1="46.95" y1="86.05" x2="42.0575" y2="86.05" width="0.4064" layer="1"/>
+<wire x1="42.0575" y1="86.05" x2="40.927" y2="84.9195" width="0.4064" layer="1"/>
 </signal>
 </signals>
