File: EscornaCPU/2.x/2.20/Escorna_CPU_2_20.brd (EAGLE design)
At the start: 50 x 100.1 mm, 105 parts, among them IC1 ULN2803, U2 ESP01, U6 ASM1117-3.3, X1 AK550/2, X1.1 AK550/2

Commit message: update
Parts:
- U6: value ASM1117-3.3 -> AMS1117-3.3
Changed lines of the file:
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@@
 <?xml version="1.0" encoding="utf-8"?>
 <!DOCTYPE eagle SYSTEM "eagle.dtd">
-<eagle version="6.4">
+<eagle version="6.5.0">
 <drawing>
 <settings>
@@
 <element name="ESC1" library="escorna" package="ESCORNA_PEQUE" value="ESCORNABOT" x="40.1955" y="55.876" smashed="yes" rot="MR0"/>
 <element name="ESC2" library="escorna" package="ESCORNA_PEQUE" value="ESCORNABOT" x="30.2" y="59.95"/>
-<element name="U6" library="Itead_IC_110429" package="SOT223" value="ASM1117-3.3" x="32.8" y="75.3"/>
+<element name="U6" library="Itead_IC_110429" package="SOT223" value="AMS1117-3.3" x="32.8" y="75.3"/>
 <element name="C1.2" library="rcl" package="C0603K" value="1uF" x="37.35" y="75.3" smashed="yes" rot="R270">
 <attribute name="NAME" x="36.85" y="73.65" size="1.016" layer="25" font="vector" rot="R270"/>
