File: EscornaCPU/2.x/2.20/Escorna_CPU_2_20.sch (EAGLE design)
At the start: 92 parts, among them IC1 ULN2803, U2 ESP01, U6 ASM1117-3.3, X1 AK550/2, X1.1 AK550/2

Commit message: Upgrade
cambios en 2.20
Parts:
- LED3.1: value Orange -> Orang
Changed lines of the file:
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@@
 <part name="LED1.1" library="led" deviceset="LED" device="CHIPLED_0603" value="Blue"/>
 <part name="LED2.1" library="led" deviceset="LED" device="CHIPLED_0603" value="Reed"/>
-<part name="LED3.1" library="led" deviceset="LED" device="CHIPLED_0603" value="Orange"/>
+<part name="LED3.1" library="led" deviceset="LED" device="CHIPLED_0603" value="Orang"/>
 <part name="LED4.1" library="led" deviceset="LED" device="CHIPLED_0603" value="Green"/>
 <part name="JP2" library="SparkFunEagle-6-6-07" deviceset="JP1E" device=""/>

Commit message: Upgrade
Resolve bug
Connections:
- net CH: no longer U2.GPIO0
Changed lines of the file:
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@@
 <net name="CH" class="0">
+<segment>
+<pinref part="R13" gate="G$1" pin="2"/>
+<label x="134.62" y="45.72" size="1.778" layer="95"/>
+<pinref part="R13.1" gate="G$1" pin="2"/>
+<wire x1="134.62" y1="48.26" x2="134.62" y2="45.72" width="0.1524" layer="91"/>
+</segment>
 <segment>
 <pinref part="U2" gate="G$1" pin="CH_PD"/>
@@
 <label x="172.72" y="48.26" size="1.778" layer="95"/>
 </segment>
-<segment>
-<pinref part="U2" gate="G$1" pin="GPIO0"/>
-<pinref part="R13" gate="G$1" pin="2"/>
-<wire x1="139.7" y1="45.72" x2="134.62" y2="45.72" width="0.1524" layer="91"/>
-<label x="137.16" y="45.72" size="1.778" layer="95"/>
-<pinref part="R13.1" gate="G$1" pin="2"/>
-<wire x1="134.62" y1="48.26" x2="134.62" y2="45.72" width="0.1524" layer="91"/>
-<junction x="134.62" y="45.72"/>
-</segment>
 </net>

Commit message: update
Parts:
- U6: value ASM1117-3.3 -> AMS1117-3.3
Changed lines of the file:
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@@
 <?xml version="1.0" encoding="utf-8"?>
 <!DOCTYPE eagle SYSTEM "eagle.dtd">
-<eagle version="6.4">
+<eagle version="6.5.0">
 <drawing>
 <settings>
@@
 <part name="H6" library="holes" deviceset="MOUNT-HOLE" device="3.0" value="H3.0"/>
 <part name="ESC2" library="escorna" deviceset="ESCORNABOT" device=""/>
-<part name="U6" library="Itead_IC_110429" deviceset="ASM1117-3.3" device=""/>
+<part name="U6" library="Itead_IC_110429" deviceset="ASM1117-3.3" device="" value="AMS1117-3.3"/>
 <part name="SUPPLY14" library="supply2" deviceset="GND" device=""/>
 <part name="C1.2" library="rcl" deviceset="C-EU" device="C0603K" value="1uF"/>
