File: EscornaCPU/2.x/2.40/Escorna_CPU_2_40Amt.brd (EAGLE design)
At the start: 50 x 90.6 mm, 112 parts, among them IC2 ULN2803, IC3 ATMEGA328P-AU, IC4 SX1308, J1 2.54, J2 10118194-0001LF/C, J3 ZL262-4SG, J5 ZL262-4SG, U1 CH340ESMD, U3 ASM1117-5.0, X1 1776275-2, X1.1 1776275-2, Y1 CSTCE16M0V53C-R0

Commit message: update
Parts:
- removed R7.1: 10K, rcl:R0603
- added R19.1: 10K, rcl:R0603
- moved R14 2.25 mm to (13.6, 44.9)
- moved R14.1 2.25 mm to (13.6, 44.9)
- moved R19 2.25 mm to (15.8, 44.9)
Connections:
- net 5V: now also R14.1, R14.1.1; no longer R19.1, R7.1.1
- net A7: now also R19.1.2; no longer R7.1.2
- net S1: now also R19.1, R19.1.1; no longer R14.1, R14.1.1
Changed lines of the file:
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@@
 <layer number="19" name="Unrouted" color="6" fill="1" visible="no" active="yes"/>
 <layer number="20" name="Dimension" color="15" fill="1" visible="yes" active="yes"/>
-<layer number="21" name="tPlace" color="7" fill="1" visible="no" active="yes"/>
+<layer number="21" name="tPlace" color="7" fill="1" visible="yes" active="yes"/>
 <layer number="22" name="bPlace" color="7" fill="1" visible="no" active="yes"/>
-<layer number="23" name="tOrigins" color="15" fill="1" visible="no" active="yes"/>
+<layer number="23" name="tOrigins" color="15" fill="1" visible="yes" active="yes"/>
 <layer number="24" name="bOrigins" color="15" fill="1" visible="no" active="yes"/>
-<layer number="25" name="tNames" color="7" fill="1" visible="no" active="yes"/>
+<layer number="25" name="tNames" color="7" fill="1" visible="yes" active="yes"/>
 <layer number="26" name="bNames" color="7" fill="1" visible="no" active="yes"/>
-<layer number="27" name="tValues" color="7" fill="1" visible="no" active="yes"/>
+<layer number="27" name="tValues" color="7" fill="1" visible="yes" active="yes"/>
 <layer number="28" name="bValues" color="7" fill="1" visible="no" active="yes"/>
 <layer number="29" name="tStop" color="7" fill="3" visible="no" active="yes"/>
 <layer number="30" name="bStop" color="7" fill="6" visible="no" active="yes"/>
-<layer number="31" name="tCream" color="7" fill="4" visible="no" active="yes"/>
+<layer number="31" name="tCream" color="7" fill="4" visible="yes" active="yes"/>
 <layer number="32" name="bCream" color="7" fill="5" visible="no" active="yes"/>
 <layer number="33" name="tFinish" color="6" fill="3" visible="no" active="yes"/>
@@
 <element name="ESC" library="escorna" package="ESCORNA_PEQUE" value="ESCORNABOT" x="27.388559375" y="22.47818125" smashed="yes" rot="MR0"/>
 <element name="XDS" library="xdesig" package="XDESIG_CU_2" value="XDESIG" x="5.86706875" y="71.35756875" smashed="yes"/>
-<element name="R14" library="rcl" package="0204/7" value="10K" x="15.8475" y="44.86" smashed="yes" rot="R90">
-<attribute name="NAME" x="12.3946" y="43.707" size="1.016" layer="25" font="vector" rot="R90"/>
-<attribute name="VALUE" x="12.9699" y="40.1156" size="1.016" layer="27" font="vector" rot="R270"/>
+<element name="R19" library="rcl" package="0204/7" value="10K" x="15.8475" y="44.86" smashed="yes" rot="R90">
+<attribute name="NAME" x="18.226234375" y="40.688303125" size="1.016" layer="25" font="vector" rot="R90"/>
+<attribute name="VALUE" x="17.330090625" y="49.2479125" size="1.016" layer="27" font="vector" rot="R270"/>
 </element>
 <element name="R15" library="rcl" package="0204/7" value="10K" x="15.856734375" y="35.808" smashed="yes" rot="R90">
@@
 <element name="H2" library="holes" package="3,0" value="3.0" x="44.2995" y="84.9465" smashed="yes"/>
 <element name="H1" library="holes" package="3,0" value="3.0" x="6.1995" y="78.5965" smashed="yes"/>
-<element name="R14.1" library="rcl" package="R0603" value="10K" x="15.8475" y="44.86" smashed="yes" rot="R90">
+<element name="R19.1" library="rcl" package="R0603" value="10K" x="15.8475" y="44.86" smashed="yes" rot="R90">
 <attribute name="NAME" x="16.3555" y="43.082" size="1.27" layer="48" rot="R90"/>
 </element>
@@
 <element name="F1.1" library="adafruit" package="R1206" value="ERF-RA05060Z" x="44.715715625" y="39.278984375" smashed="yes" rot="R270"/>
 <element name="$1_82_$" library="Escorna_CPU_2_01" package="XDESIG_XDESIG" value="XDESIG_XDESIG21" x="27.53888125" y="48.765778125" rot="MR0"/>
-<element name="R7.1" library="rcl" package="R0603" value="10K" x="13.5975" y="44.86" smashed="yes" rot="R90">
+<element name="R14.1" library="rcl" package="R0603" value="10K" x="13.5975" y="44.86" smashed="yes" rot="R90">
 <attribute name="NAME" x="14.1055" y="43.082" size="1.27" layer="48" rot="R90"/>
 </element>
-<element name="R19" library="rcl" package="0204/7" value="10K" x="13.5975" y="44.86" smashed="yes" rot="R90">
-<attribute name="NAME" x="17.2054" y="43.343" size="1.016" layer="25" font="vector" rot="R270"/>
-<attribute name="VALUE" x="17.2199" y="48.7656" size="1.016" layer="27" font="vector" rot="R270"/>
+<element name="R14" library="rcl" package="0204/7" value="10K" x="13.5975" y="44.86" smashed="yes" rot="R90">
+<attribute name="NAME" x="12.26566875" y="43.81171875" size="1.016" layer="25" font="vector" rot="R90"/>
+<attribute name="VALUE" x="12.9551875" y="40.141009375" size="1.016" layer="27" font="vector" rot="R270"/>
 </element>
 <element name="R8" library="rcl" package="0204/7" value="1K" x="34.24164375" y="39.15" smashed="yes" rot="R270">
@@
 </signal>
 <signal name="A7">
+<contactref element="R14" pad="2"/>
+<contactref element="IC3" pad="22"/>
+<contactref element="R19.1" pad="2"/>
 <contactref element="R19" pad="2"/>
-<contactref element="IC3" pad="22"/>
+<wire x1="15.8475" y1="45.71" x2="15.8475" y2="48.67" width="0.8128" layer="1"/>
 <contactref element="R14.1" pad="2"/>
-<contactref element="R14" pad="2"/>
-<wire x1="15.8475" y1="45.71" x2="15.8475" y2="48.67" width="0.8128" layer="1"/>
-<contactref element="R7.1" pad="2"/>
 <wire x1="16.0074" y1="62.7" x2="14.2" y2="62.7" width="0.4064" layer="1"/>
 <wire x1="15.8475" y1="48.67" x2="13.5975" y2="48.67" width="0.8128" layer="16"/>
@@
 <signal name="S1">
 <contactref element="R15" pad="2"/>
-<contactref element="R14" pad="1"/>
-<contactref element="R14.1" pad="1"/>
+<contactref element="R19" pad="1"/>
+<contactref element="R19.1" pad="1"/>
 <contactref element="R15.1" pad="2"/>
 <wire x1="15.857265625" y1="36.65310625" x2="15.856734375" y2="39.618" width="0.8128" layer="1"/>
@@
 <contactref element="IC3" pad="6"/>
 <contactref element="R7" pad="1"/>
-<contactref element="R19" pad="1"/>
+<contactref element="R14" pad="1"/>
 <contactref element="ICSP" pad="2"/>
 <contactref element="C7" pad="1"/>
@@
 <wire x1="14.439" y1="65.9" x2="16.0074" y2="65.9" width="0.3048" layer="1"/>
 <contactref element="J5" pad="4"/>
-<contactref element="R7.1" pad="1"/>
+<contactref element="R14.1" pad="1"/>
 <contactref element="J3" pad="3"/>
 <wire x1="24.5926" y1="65.1" x2="23.204675" y2="65.1" width="0.4064" layer="1"/>

Commit message: Update
Parts:
- removed XDS2: XDESIG, xdesig:XDESIG_CU_2
- moved XDS1 35.6 mm to (26.2, 40.6)
- moved $1_82_$ 9.36 mm to (27.5, 39.4)
- moved R14 2.25 mm to (15.8, 44.9)
- moved R14.1 2.25 mm to (15.8, 44.9)
- moved R19 2.25 mm to (13.6, 44.9)
- moved R19.1 2.25 mm to (13.6, 44.9)
Connections:
- net 5V: now also R19.1, R19.1.1; no longer R14.1, R14.1.1
- net S1: now also R14.1, R14.1.1; no longer R19.1, R19.1.1
Routing:
- net D10: track 62.2 -> 43.7 mm
- net RAW: track 82.9 -> 85.9 mm
- net GND: vias 31 -> 36
Other:
- board text added: "2042"
- board text added: "CPU 2.40.1"
- board text added: "OSHWA ES11"
- board text removed: "2011"
