File: EscornaCPU/2.x/2.40/Escorna_CPU_2_40Amt.sch (EAGLE design)
At the start: 101 parts, among them IC2 ULN2803, IC3 ATMEGA328P-AU, IC4 SX1308, J1 2.54, J2 10118194-0001LF/C, J3 ZL262-4SG, J5 ZL262-4SG, U1 CH340ESMD, U3 ASM1117-5.0, X1 1776275-2, X1.1 1776275-2, Y1 CSTCE16M0V53C-R0

Commit message: update
Parts:
- removed R7.1: 10K, rcl:R-EU_R0603
- added R19.1: 10K, rcl:R-EU_R0603
Connections:
- net 5V: now also R14.1, R14.1.1; no longer R19.1, R7.1.1
- net A7: now also R19.1.2; no longer R7.1.2
- net S1: now also R19.1, R19.1.1; no longer R14.1, R14.1.1
Other:
- note added: "002"
- note removed: "001"
- moved on the sheet: R14, R14.1, R19
Changed lines of the file:
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@@
 <part name="XDS2" library="xdesig" deviceset="XDESIG" device=""/>
 <part name="ESC" library="escorna" deviceset="ESCORNABOT" device=""/>
-<part name="R14" library="rcl" deviceset="R-EU_" device="0204/7" value="10K"/>
+<part name="R19" library="rcl" deviceset="R-EU_" device="0204/7" value="10K"/>
 <part name="R15" library="rcl" deviceset="R-EU_" device="0204/7" value="10K"/>
 <part name="R16" library="rcl" deviceset="R-EU_" device="0204/7" value="10K"/>
@@
 <part name="H2" library="holes" deviceset="MOUNT-HOLE" device="3.0" value="3.0"/>
 <part name="H1" library="holes" deviceset="MOUNT-HOLE" device="3.0" value="3.0"/>
-<part name="R14.1" library="rcl" deviceset="R-EU_" device="R0603" value="10K"/>
+<part name="R19.1" library="rcl" deviceset="R-EU_" device="R0603" value="10K"/>
 <part name="R15.1" library="rcl" deviceset="R-EU_" device="R0603" value="10K"/>
 <part name="R16.1" library="rcl" deviceset="R-EU_" device="R0603" value="10K"/>
@@
 </part>
 <part name="F1.1" library="adafruit" deviceset="PTCFUSE" device="-1206" value="ERF-RA05060Z"/>
-<part name="R7.1" library="rcl" deviceset="R-EU_" device="R0603" value="10K"/>
-<part name="R19" library="rcl" deviceset="R-EU_" device="0204/7" value="10K"/>
+<part name="R14.1" library="rcl" deviceset="R-EU_" device="R0603" value="10K"/>
+<part name="R14" library="rcl" deviceset="R-EU_" device="0204/7" value="10K"/>
 <part name="R8" library="rcl" deviceset="R-EU_" device="0204/7" value="1K"/>
 <part name="R9" library="rcl" deviceset="R-EU_" device="0204/7" value="1K"/>
@@
 <text x="246.888" y="17.526" size="1.778" layer="97">XDeSIG</text>
 <text x="173.228" y="25.4" size="2.54" layer="97">PseudoSingularis (PSingularis)  by XDeSIG.</text>
-<text x="254" y="7.62" size="2.54" layer="97">001</text>
+<text x="254" y="7.62" size="2.54" layer="97">002</text>
 <text x="221.234" y="132.334" size="2.54" layer="95">Enabling LEDs, Default on</text>
 <text x="159.766" y="77.978" size="1.778" layer="97" rot="R270">BUZZ on/off</text>
@@
 <instance part="XDS2" gate="G$1" x="259.08" y="17.78"/>
 <instance part="ESC" gate="G$1" x="132.08" y="86.36"/>
-<instance part="R14" gate="G$1" x="195.58" y="162.56" rot="R180"/>
+<instance part="R19" gate="G$1" x="195.58" y="162.56" rot="R180"/>
 <instance part="R15" gate="G$1" x="208.28" y="162.56" rot="R180"/>
 <instance part="R16" gate="G$1" x="220.98" y="162.56" rot="R180"/>
@@
 <instance part="H2" gate="G$1" x="2.54" y="53.34"/>
 <instance part="H1" gate="G$1" x="2.54" y="45.72"/>
-<instance part="R14.1" gate="G$1" x="195.58" y="170.18" rot="R180"/>
+<instance part="R19.1" gate="G$1" x="195.58" y="170.18" rot="R180"/>
 <instance part="R15.1" gate="G$1" x="208.28" y="170.18" rot="R180"/>
 <instance part="R16.1" gate="G$1" x="220.98" y="170.18" rot="R180"/>
@@
 <attribute name="NAME" x="21.59" y="27.94" size="1.778" layer="95"/>
 </instance>
-<instance part="R7.1" gate="G$1" x="185.42" y="167.64" rot="R270"/>
-<instance part="R19" gate="G$1" x="177.8" y="167.64" rot="R270"/>
+<instance part="R14.1" gate="G$1" x="185.42" y="167.64" rot="R270"/>
+<instance part="R14" gate="G$1" x="177.8" y="167.64" rot="R270"/>
 <instance part="R8" gate="G$1" x="203.2" y="111.76" rot="R270"/>
 <instance part="R9" gate="G$1" x="220.98" y="111.76" rot="R270"/>
@@
 <label x="172.72" y="162.56" size="1.778" layer="95"/>
 <wire x1="177.8" y1="162.56" x2="172.72" y2="162.56" width="0.1524" layer="91"/>
+<pinref part="R14" gate="G$1" pin="2"/>
 <pinref part="R19" gate="G$1" pin="2"/>
-<pinref part="R14" gate="G$1" pin="2"/>
-<pinref part="R14.1" gate="G$1" pin="2"/>
+<pinref part="R19.1" gate="G$1" pin="2"/>
 <wire x1="190.5" y1="170.18" x2="190.5" y2="162.56" width="0.1524" layer="91"/>
 <wire x1="190.5" y1="162.56" x2="185.42" y2="162.56" width="0.1524" layer="91"/>
@@
 <wire x1="185.42" y1="162.56" x2="177.8" y2="162.56" width="0.1524" layer="91"/>
 <junction x="185.42" y="162.56"/>
-<pinref part="R7.1" gate="G$1" pin="2"/>
+<pinref part="R14.1" gate="G$1" pin="2"/>
 </segment>
 <segment>
@@
 <segment>
 <pinref part="R15" gate="G$1" pin="2"/>
-<pinref part="R14" gate="G$1" pin="1"/>
+<pinref part="R19" gate="G$1" pin="1"/>
 <wire x1="203.2" y1="162.56" x2="200.66" y2="162.56" width="0.1524" layer="91"/>
 <wire x1="203.2" y1="160.02" x2="203.2" y2="162.56" width="0.1524" layer="91"/>
 <junction x="203.2" y="162.56"/>
-<pinref part="R14.1" gate="G$1" pin="1"/>
+<pinref part="R19.1" gate="G$1" pin="1"/>
 <pinref part="R15.1" gate="G$1" pin="2"/>
 <wire x1="200.66" y1="170.18" x2="203.2" y2="170.18" width="0.1524" layer="91"/>
@@
 </segment>
 <segment>
-<pinref part="R19" gate="G$1" pin="1"/>
+<pinref part="R14" gate="G$1" pin="1"/>
 <wire x1="185.42" y1="172.72" x2="177.8" y2="172.72" width="0.1524" layer="91"/>
-<pinref part="R7.1" gate="G$1" pin="1"/>
+<pinref part="R14.1" gate="G$1" pin="1"/>
 <pinref part="U$18" gate="G$1" pin="5V"/>
 <junction x="177.8" y="172.72"/>

Commit message: Update
Parts:
- removed XDS2: XDESIG, xdesig:XDESIG
Connections:
- net 5V: now also R19.1, R19.1.1; no longer R14.1, R14.1.1
- net S1: now also R14.1, R14.1.1; no longer R19.1, R19.1.1
Other:
- note removed: "Amtega Logo"
- moved on the sheet: R14, R14.1, R19, R19.1
Changed lines of the file:
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@@
 <part name="H3" library="holes" deviceset="MOUNT-HOLE" device="3.0" value="3.0"/>
 <part name="H4" library="holes" deviceset="MOUNT-HOLE" device="3.0" value="3.0"/>
-<part name="XDS2" library="xdesig" deviceset="XDESIG" device=""/>
 <part name="ESC" library="escorna" deviceset="ESCORNABOT" device=""/>
-<part name="R19" library="rcl" deviceset="R-EU_" device="0204/7" value="10K"/>
+<part name="R14" library="rcl" deviceset="R-EU_" device="0204/7" value="10K"/>
 <part name="R15" library="rcl" deviceset="R-EU_" device="0204/7" value="10K"/>
 <part name="R16" library="rcl" deviceset="R-EU_" device="0204/7" value="10K"/>
@@
 <part name="H2" library="holes" deviceset="MOUNT-HOLE" device="3.0" value="3.0"/>
 <part name="H1" library="holes" deviceset="MOUNT-HOLE" device="3.0" value="3.0"/>
-<part name="R19.1" library="rcl" deviceset="R-EU_" device="R0603" value="10K"/>
+<part name="R14.1" library="rcl" deviceset="R-EU_" device="R0603" value="10K"/>
 <part name="R15.1" library="rcl" deviceset="R-EU_" device="R0603" value="10K"/>
 <part name="R16.1" library="rcl" deviceset="R-EU_" device="R0603" value="10K"/>
@@
 </part>
 <part name="F1.1" library="adafruit" deviceset="PTCFUSE" device="-1206" value="ERF-RA05060Z"/>
-<part name="R14.1" library="rcl" deviceset="R-EU_" device="R0603" value="10K"/>
-<part name="R14" library="rcl" deviceset="R-EU_" device="0204/7" value="10K"/>
+<part name="R19.1" library="rcl" deviceset="R-EU_" device="R0603" value="10K"/>
+<part name="R19" library="rcl" deviceset="R-EU_" device="0204/7" value="10K"/>
 <part name="R8" library="rcl" deviceset="R-EU_" device="0204/7" value="1K"/>
 <part name="R9" library="rcl" deviceset="R-EU_" device="0204/7" value="1K"/>
@@
 <text x="88.646" y="37.338" size="2.54" layer="95" rot="R180">Step-up power</text>
 <text x="75.184" y="4.572" size="1.778" layer="97">MT3608</text>
-<text x="88.9" y="96.52" size="2.54" layer="97" align="center">
-Amtega
-Logo
-</text>
 </plain>
 <instances>
@@
 <instance part="H3" gate="G$1" x="2.54" y="60.96"/>
 <instance part="H4" gate="G$1" x="2.54" y="68.58"/>
-<instance part="XDS2" gate="G$1" x="259.08" y="17.78"/>
 <instance part="ESC" gate="G$1" x="132.08" y="86.36"/>
-<instance part="R19" gate="G$1" x="195.58" y="162.56" rot="R180"/>
+<instance part="R14" gate="G$1" x="195.58" y="162.56" rot="R180"/>
 <instance part="R15" gate="G$1" x="208.28" y="162.56" rot="R180"/>
 <instance part="R16" gate="G$1" x="220.98" y="162.56" rot="R180"/>
@@
 <instance part="H2" gate="G$1" x="2.54" y="53.34"/>
 <instance part="H1" gate="G$1" x="2.54" y="45.72"/>
-<instance part="R19.1" gate="G$1" x="195.58" y="170.18" rot="R180"/>
+<instance part="R14.1" gate="G$1" x="195.58" y="170.18" rot="R180"/>
 <instance part="R15.1" gate="G$1" x="208.28" y="170.18" rot="R180"/>
 <instance part="R16.1" gate="G$1" x="220.98" y="170.18" rot="R180"/>
@@
 <attribute name="NAME" x="21.59" y="27.94" size="1.778" layer="95"/>
 </instance>
-<instance part="R14.1" gate="G$1" x="185.42" y="167.64" rot="R270"/>
-<instance part="R14" gate="G$1" x="177.8" y="167.64" rot="R270"/>
+<instance part="R19.1" gate="G$1" x="185.42" y="167.64" rot="R270"/>
+<instance part="R19" gate="G$1" x="177.8" y="167.64" rot="R270"/>
 <instance part="R8" gate="G$1" x="203.2" y="111.76" rot="R270"/>
 <instance part="R9" gate="G$1" x="220.98" y="111.76" rot="R270"/>
@@
 <label x="172.72" y="162.56" size="1.778" layer="95"/>
 <wire x1="177.8" y1="162.56" x2="172.72" y2="162.56" width="0.1524" layer="91"/>
+<pinref part="R19" gate="G$1" pin="2"/>
 <pinref part="R14" gate="G$1" pin="2"/>
-<pinref part="R19" gate="G$1" pin="2"/>
-<pinref part="R19.1" gate="G$1" pin="2"/>
+<pinref part="R14.1" gate="G$1" pin="2"/>
 <wire x1="190.5" y1="170.18" x2="190.5" y2="162.56" width="0.1524" layer="91"/>
 <wire x1="190.5" y1="162.56" x2="185.42" y2="162.56" width="0.1524" layer="91"/>
@@
 <wire x1="185.42" y1="162.56" x2="177.8" y2="162.56" width="0.1524" layer="91"/>
 <junction x="185.42" y="162.56"/>
-<pinref part="R14.1" gate="G$1" pin="2"/>
+<pinref part="R19.1" gate="G$1" pin="2"/>
 </segment>
 <segment>
@@
 <segment>
 <pinref part="R15" gate="G$1" pin="2"/>
-<pinref part="R19" gate="G$1" pin="1"/>
+<pinref part="R14" gate="G$1" pin="1"/>
 <wire x1="203.2" y1="162.56" x2="200.66" y2="162.56" width="0.1524" layer="91"/>
 <wire x1="203.2" y1="160.02" x2="203.2" y2="162.56" width="0.1524" layer="91"/>
 <junction x="203.2" y="162.56"/>
-<pinref part="R19.1" gate="G$1" pin="1"/>
+<pinref part="R14.1" gate="G$1" pin="1"/>
 <pinref part="R15.1" gate="G$1" pin="2"/>
 <wire x1="200.66" y1="170.18" x2="203.2" y2="170.18" width="0.1524" layer="91"/>
@@
 </segment>
 <segment>
-<pinref part="R14" gate="G$1" pin="1"/>
+<pinref part="R19" gate="G$1" pin="1"/>
 <wire x1="185.42" y1="172.72" x2="177.8" y2="172.72" width="0.1524" layer="91"/>
-<pinref part="R14.1" gate="G$1" pin="1"/>
+<pinref part="R19.1" gate="G$1" pin="1"/>
 <pinref part="U$18" gate="G$1" pin="5V"/>
 <junction x="177.8" y="172.72"/>
